File: doc/shuttersKicad/shutters.kicad_pcb (KiCad board)
At the start: 2 copper layers, 140 parts, among them J1 Conn_02x05_Top_Bottom, J10 Screw_Terminal_01x08, J11 Screw_Terminal_01x08, J12 Screw_Terminal_01x08, J2 Screw_Terminal_01x08, J3 Screw_Terminal_01x08, J4 Screw_Terminal_01x02, J5 Screw_Terminal_01x08, J6 Screw_Terminal_01x08, J7 Screw_Terminal_01x02, J8 Screw_Terminal_01x08, J9 Screw_Terminal_01x08, Q1 BSS138, Q10 BSS138, Q2 BSS138, Q3 BSS138, Q4 BSS138, Q5 BSS138, Q6 BSS138, Q7 BSS138, Q8 BSS138, Q9 BSS138, SW1 SW_DIP_x03, SW2 SW_DIP_x03, SW3 SW_DIP_x03, SW4 SW_DIP_x03, U1 ESP32-DEVKITC, U10 SFH617A-1X006, U11 SFH617A-1X006, U12 SFH617A-1X006, U13 SFH617A-1X006, U14 SFH617A-1X006, U15 SFH617A-1X006, U16 SFH617A-1X006, U17 SFH617A-1X006, U18 MCP23017_SP, U19 SFH617A-1X006, U2 SFH617A-1X006, U20 SFH617A-1X006, U21 SFH617A-1X006, U22 SFH617A-1X006, U23 SFH617A-1X006, U24 SFH617A-1X006, U25 SFH617A-1X006, U26 SFH617A-1X006, U27 SFH617A-1X006, U28 SFH617A-1X006, U29 SFH617A-1X006, U3 SFH617A-1X006, U30 SFH617A-1X006, U31 SFH617A-1X006, U32 SFH617A-1X006, U33 SFH617A-1X006, U34 SFH617A-1X006, U35 MCP23017_SP, U36 MCP23017_SP, U37 MCP23017_SP, U38 ULN2003A, U39 ULN2003A, U4 SFH617A-1X006, U40 ULN2003A, U41 ULN2003A, U42 ULN2003A, U5 SFH617A-1X006, U6 SFH617A-1X006, U7 SFH617A-1X006, U8 SFH617A-1X006, U9 SFH617A-1X006

Commit message: edit kicad
Parts:
- removed J12, J9: Screw_Terminal_01x08, TerminalBlock_Phoenix:TerminalBlock_Phoenix_MKDS-1,5-8-5.08_1x08_P5.08mm_Horizontal
- removed Q1, Q10, Q2, Q3, Q4, Q5, Q6, Q7, Q8, Q9: BSS138, Package_TO_SOT_THT:TO-92L_HandSolder
- removed R10, R11, R12, R13, R14, R15, R16, R40, R41, R42, R43, R44, R45, R46, R47, R48, R49, R5, R50, R51, R52, R53, R54, R55, R6, R7, R8, R9: 560, Resistor_THT:R_Axial_DIN0204_L3.6mm_D1.6mm_P5.08mm_Horizontal
- removed R17, R18, R19, R20, R21, R22, R23, R24, R25, R26, R27, R28, R29, R30, R31, R33, R35, R36, R38, R39: 10k, Resistor_THT:R_Axial_DIN0204_L3.6mm_D1.6mm_P5.08mm_Horizontal
- removed R32, R34, R37, R56, R57, R58, R59, R60, R61, R62, R63, R64: 10K, Resistor_THT:R_Axial_DIN0204_L3.6mm_D1.6mm_P5.08mm_Horizontal
- removed SW1, SW2, SW3, SW4: SW_DIP_x03, Button_Switch_THT:SW_DIP_SPSTx03_Slide_9.78x9.8mm_W7.62mm_P2.54mm
- removed U10, U11, U12, U13, U14, U15, U16, U17, U19, U20, U21, U22, U23, U24, U25, U26, U27, U28, U29, U30, U31, U32, U33, U34, U5, U6, U7, U8, U9: SFH617A-1X006, Package_DIP:DIP-4_W10.16mm
- removed U35: MCP23017_SP, Package_DIP:DIP-28_W7.62mm
- removed U38, U40: ULN2003A, Package_DIP:DIP-16_W7.62mm_Socket
- added J13: Pin Header_01x10, Connector_PinHeader_2.54mm:PinHeader_1x10_P2.54mm_Vertical, F.Cu at (67.8, 68.6)
- added J14: Pin Header_01x10, Connector_PinHeader_2.54mm:PinHeader_1x10_P2.54mm_Vertical, F.Cu at (54.8, 68.6)
- added J15: Pin Header_01x10, Connector_PinHeader_2.54mm:PinHeader_1x10_P2.54mm_Vertical, F.Cu at (87.9, 68.5)
- added J16: Pin Header_01x10, Connector_PinHeader_2.54mm:PinHeader_1x10_P2.54mm_Vertical, F.Cu at (74.9, 68.5)
- added JP1: Jumper_2_Open, Connector_PinHeader_2.54mm:PinHeader_1x02_P2.54mm_Vertical, F.Cu at (23.9, 63.2)
- added JP2: Jumper_2_Open, Connector_PinHeader_2.54mm:PinHeader_1x02_P2.54mm_Vertical, F.Cu at (18.9, 90.6)
- added JP3: Jumper_2_Open, Connector_PinHeader_2.54mm:PinHeader_1x02_P2.54mm_Vertical, F.Cu at (45.9, 43.7)
- added JP4: Jumper_2_Open, Connector_PinHeader_2.54mm:PinHeader_1x02_P2.54mm_Vertical, F.Cu at (83.9, 40.9)
- J7: value Screw_Terminal_01x02 -> Screw_Terminal_01x08; footprint TerminalBlock_Phoenix:TerminalBlock_Phoenix_MKDS-1,5-2-5.08_1x02_P5.08mm_Horizontal -> TerminalBlock_Phoenix:TerminalBlock_Phoenix_MKDS-1,5-8-5.08_1x08_P5.08mm_Horizontal
- R1, R2, R3, R4: value 560 -> 10K
- U2: value SFH617A-1X006 -> MCP23017_SP; footprint Package_DIP:DIP-4_W10.16mm -> Package_DIP:DIP-28_W7.62mm
- U3, U4: value SFH617A-1X006 -> ULN2003A; footprint Package_DIP:DIP-4_W10.16mm -> Package_DIP:DIP-16_W7.62mm_Socket
- moved H3 205.2 mm to (6.47, 100.7)
- moved H1 202.8 mm to (8.03, 5.70)
- moved U3 190.5 mm to (21.9, 23.9), turned to 90 degrees
- moved R1 181.4 mm to (84.2, 68.6), turned to 90 degrees
- moved R2 177.9 mm to (80.8, 68.5), turned to 90 degrees
- moved U4 161.2 mm to (75.0, 23.0), turned to 90 degrees
- moved J3 148.0 mm to (6.50, 56.8), turned to -90 degrees
- moved R4 146.4 mm to (79.9, 54.6), turned to -90 degrees
- moved J8 144.5 mm to (56.4, 6.12), turned to 180 degrees
- moved R3 142.6 mm to (83.2, 54.6), turned to -90 degrees
- moved J7 136.7 mm to (100.5, 6.22), turned to 180 degrees
- moved U2 135.8 mm to (51.6, 76.2), turned to -90 degrees
- moved U39 128.9 mm to (46.2, 23.7), turned to 90 degrees
- moved H2 123.6 mm to (132.0, 16.9)
- moved U36 115.4 mm to (62.2, 30.6), turned to -90 degrees
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Connections:
- J1 pad 1: +3V3 -> unconnected-(J1-Pad1)
- J1 pad 2: GND -> Net-(J1-Pad2)
- J1 pad 3: GND -> Net-(J1-Pad2)
- J1 pad 4: GND -> Net-(J1-Pad2)
- J1 pad 5: GND -> Net-(J1-Pad2)
- J10 pad 8: +5V -> Net-(J10-Pad8)
- J11 pad 8: +5V -> Net-(J11-Pad8)
- J4 pad 1: unconnected-(J4-Pad1) -> +5V
- J4 pad 2: unconnected-(J4-Pad2) -> GND
- J7 pad 1: +5V -> Net-(J7-Pad1)
- J7 pad 2: GND -> Net-(J7-Pad2)
- J8 pad 8: +5V -> Net-(J8-Pad8)
- R1 pad 1: Net-(J2-Pad1) -> +3V3
- R1 pad 2: Net-(R1-Pad2) -> Net-(J15-Pad2)
- R2 pad 1: Net-(J2-Pad2) -> +3V3
- R2 pad 2: Net-(R2-Pad2) -> Net-(J15-Pad3)
- R3 pad 1: Net-(J2-Pad3) -> +5V
- R3 pad 2: Net-(R3-Pad2) -> Net-(J16-Pad2)
- R4 pad 1: Net-(J2-Pad4) -> +5V
- R4 pad 2: Net-(R4-Pad2) -> Net-(J16-Pad3)
- U1 pad 25: Net-(Q1-Pad2) -> unconnected-(U1-Pad25)
- U1 pad 26: Net-(Q2-Pad2) -> unconnected-(U1-Pad26)
- U1 pad 27: Net-(Q3-Pad2) -> unconnected-(U1-Pad27)
- U1 pad 29: Net-(Q6-Pad2) -> unconnected-(U1-Pad29)
- U1 pad 33: Net-(Q7-Pad2) -> Net-(J15-Pad2)
- U1 pad 36: Net-(Q8-Pad2) -> Net-(J15-Pad3)
- U18 pad 1: Net-(U18-Pad1) -> Net-(J2-Pad1)
- U18 pad 12: /I2C-SCL-5V -> Net-(J16-Pad3)
- U18 pad 13: /I2C-SDA-5V -> Net-(J16-Pad2)
- U18 pad 15: Net-(R37-Pad1) -> +5V
- U18 pad 16: Net-(R34-Pad1) -> +5V
- U18 pad 17: Net-(R32-Pad1) -> +5V
- U18 pad 2: Net-(U18-Pad2) -> Net-(J2-Pad2)
- U18 pad 21: Net-(U10-Pad4) -> Net-(J3-Pad1)
- U18 pad 22: Net-(U11-Pad4) -> Net-(J3-Pad2)
- U18 pad 23: Net-(U12-Pad4) -> Net-(J3-Pad3)
- U18 pad 24: Net-(U13-Pad4) -> Net-(J3-Pad4)
- U18 pad 25: Net-(U14-Pad4) -> Net-(J3-Pad5)
- U18 pad 26: Net-(U15-Pad4) -> Net-(J3-Pad6)
- U18 pad 27: Net-(U16-Pad4) -> Net-(J3-Pad7)
- U18 pad 28: Net-(U17-Pad4) -> Net-(J3-Pad8)
- U18 pad 3: Net-(U18-Pad3) -> Net-(J2-Pad3)
- U18 pad 4: Net-(U18-Pad4) -> Net-(J2-Pad4)
- U18 pad 5: Net-(U18-Pad5) -> Net-(J2-Pad5)
- U18 pad 6: Net-(U18-Pad6) -> Net-(J2-Pad6)
- U18 pad 7: Net-(U18-Pad7) -> Net-(J2-Pad7)
- U18 pad 8: Net-(U18-Pad8) -> Net-(J2-Pad8)
- U2 pad 1: Net-(R1-Pad2) -> Net-(J5-Pad8)
- U2 pad 2: GND -> Net-(J5-Pad7)
- U2 pad 3: GND -> Net-(J5-Pad6)
- U2 pad 4: Net-(U18-Pad1) -> Net-(J5-Pad5)
- U3 pad 1: Net-(R2-Pad2) -> Net-(U3-Pad1)
- U3 pad 2: GND -> Net-(U3-Pad2)
- U3 pad 3: GND -> Net-(U3-Pad3)
- U3 pad 4: Net-(U18-Pad2) -> Net-(U3-Pad4)
- U36 pad 1: Net-(U36-Pad1) -> Net-(U3-Pad7)
- U36 pad 12: /I2C-SCL-5V -> Net-(J16-Pad3)
- U36 pad 13: /I2C-SDA-5V -> Net-(J16-Pad2)
- U36 pad 15: Net-(R59-Pad1) -> GND
- U36 pad 16: Net-(R61-Pad1) -> GND
- U36 pad 17: Net-(R63-Pad1) -> +5V
- U36 pad 2: Net-(U36-Pad2) -> Net-(U3-Pad6)
- U36 pad 3: Net-(U36-Pad3) -> Net-(U3-Pad5)
- U36 pad 4: Net-(U36-Pad4) -> Net-(U3-Pad4)
- U36 pad 5: Net-(U36-Pad5) -> Net-(U3-Pad3)
- U36 pad 6: Net-(U36-Pad6) -> Net-(U3-Pad2)
- U36 pad 7: Net-(U36-Pad7) -> Net-(U3-Pad1)
- U37 pad 12: /I2C-SCL-5V -> Net-(J16-Pad3)
- U37 pad 13: /I2C-SDA-5V -> Net-(J16-Pad2)
- U37 pad 15: Net-(R60-Pad1) -> GND
- U37 pad 16: Net-(R62-Pad1) -> GND
- U37 pad 17: Net-(R64-Pad1) -> GND
- U39 pad 10: Net-(J9-Pad7) -> Net-(J7-Pad3)
- U39 pad 11: Net-(J9-Pad6) -> Net-(J7-Pad4)
- U39 pad 12: Net-(J9-Pad5) -> Net-(J7-Pad5)
- U39 pad 13: Net-(J9-Pad4) -> Net-(J7-Pad6)
- U39 pad 14: Net-(J9-Pad3) -> Net-(J7-Pad7)
- U39 pad 15: Net-(J9-Pad2) -> Net-(J7-Pad8)
- U39 pad 16: Net-(J9-Pad1) -> Net-(J8-Pad8)
- U4 pad 1: Net-(R3-Pad2) -> Net-(U37-Pad5)
- U4 pad 2: GND -> Net-(U37-Pad4)
- U4 pad 3: GND -> Net-(U37-Pad3)
- U4 pad 4: Net-(U18-Pad3) -> Net-(U37-Pad2)
- U41 pad 1: Net-(U37-Pad6) -> Net-(U37-Pad8)
- U41 pad 10: Net-(J11-Pad7) -> Net-(J11-Pad4)
- U41 pad 11: Net-(J11-Pad6) -> Net-(J11-Pad3)
- U41 pad 12: Net-(J11-Pad5) -> Net-(J11-Pad2)
- U41 pad 13: Net-(J11-Pad4) -> Net-(J11-Pad1)
- U41 pad 14: Net-(J11-Pad3) -> Net-(J10-Pad6)
- U41 pad 15: Net-(J11-Pad2) -> Net-(J10-Pad7)
- U41 pad 16: Net-(J11-Pad1) -> Net-(J10-Pad8)
- U41 pad 3: Net-(U37-Pad8) -> Net-(U37-Pad6)
- U42 pad 1: Net-(U37-Pad25) -> Net-(U37-Pad28)
- U42 pad 10: Net-(J12-Pad7) -> unconnected-(U42-Pad10)
- U42 pad 11: Net-(J12-Pad6) -> unconnected-(U42-Pad11)
- U42 pad 12: Net-(J12-Pad5) -> unconnected-(U42-Pad12)
- U42 pad 13: Net-(J12-Pad4) -> Net-(J11-Pad8)
- U42 pad 14: Net-(J12-Pad3) -> Net-(J11-Pad7)
- U42 pad 15: Net-(J12-Pad2) -> Net-(J11-Pad6)
- U42 pad 16: Net-(J12-Pad1) -> Net-(J11-Pad5)
- U42 pad 2: Net-(U37-Pad26) -> Net-(U37-Pad27)
- U42 pad 3: Net-(U37-Pad27) -> Net-(U37-Pad26)
- U42 pad 4: Net-(U37-Pad28) -> Net-(U37-Pad25)
Routing:
- net +5V: track 0.00 -> 502.2 mm
- net Net-(J16-Pad2): track 0.00 -> 151.7 mm
- net Net-(J16-Pad3): track 0.00 -> 147.7 mm
- net +3V3: track 0.00 -> 92.6 mm
- net Net-(J10-Pad1): track 0.00 -> 63.4 mm
- net Net-(J11-Pad1): track 0.00 -> 63.0 mm
- net Net-(J10-Pad2): track 0.00 -> 60.8 mm
- net Net-(J2-Pad1): track 0.00 -> 60.2 mm
- net Net-(J10-Pad3): track 0.00 -> 58.3 mm
- net Net-(J16-Pad5): track 0.00 -> 57.2 mm
- net Net-(J3-Pad8): track 0.00 -> 56.8 mm
- net Net-(J10-Pad4): track 0.00 -> 55.7 mm
- net Net-(J2-Pad2): track 0.00 -> 54.2 mm
- net Net-(J11-Pad2): track 0.00 -> 53.9 mm
- net Net-(J16-Pad4): track 0.00 -> 53.7 mm
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- added copper zone on B.Cu, net GND
Other:
- board outline added: 148 x 105 mm
