File: doc/shuttersKicad/shutters.kicad_sch (KiCad schematic)
At the start: 140 parts, among them J1 Conn_02x05_Top_Bottom, J10 Screw_Terminal_01x08, J11 Screw_Terminal_01x08, J12 Screw_Terminal_01x08, J2 Screw_Terminal_01x08, J3 Screw_Terminal_01x08, J4 Screw_Terminal_01x02, J5 Screw_Terminal_01x08, J6 Screw_Terminal_01x08, J7 Screw_Terminal_01x02, J8 Screw_Terminal_01x08, J9 Screw_Terminal_01x08, Q1 BSS138, Q10 BSS138, Q2 BSS138, Q3 BSS138, Q4 BSS138, Q5 BSS138, Q6 BSS138, Q7 BSS138, Q8 BSS138, Q9 BSS138, SW1 SW_DIP_x03, SW2 SW_DIP_x03, SW3 SW_DIP_x03, SW4 SW_DIP_x03, U1 ESP32-DEVKITC, U10 SFH617A-1X006, U11 SFH617A-1X006, U12 SFH617A-1X006, U13 SFH617A-1X006, U14 SFH617A-1X006, U15 SFH617A-1X006, U16 SFH617A-1X006, U17 SFH617A-1X006, U18 MCP23017_SP, U19 SFH617A-1X006, U2 SFH617A-1X006, U20 SFH617A-1X006, U21 SFH617A-1X006, U22 SFH617A-1X006, U23 SFH617A-1X006, U24 SFH617A-1X006, U25 SFH617A-1X006, U26 SFH617A-1X006, U27 SFH617A-1X006, U28 SFH617A-1X006, U29 SFH617A-1X006, U3 SFH617A-1X006, U30 SFH617A-1X006, U31 SFH617A-1X006, U32 SFH617A-1X006, U33 SFH617A-1X006, U34 SFH617A-1X006, U35 MCP23017_SP, U36 MCP23017_SP, U37 MCP23017_SP, U38 ULN2003A, U39 ULN2003A, U4 SFH617A-1X006, U40 ULN2003A, U41 ULN2003A, U42 ULN2003A, U5 SFH617A-1X006, U6 SFH617A-1X006, U7 SFH617A-1X006, U8 SFH617A-1X006, U9 SFH617A-1X006

Commit message: edit kicad
Parts:
- removed J12, J9: Screw_Terminal_01x08, TerminalBlock_Phoenix:TerminalBlock_Phoenix_MKDS-1,5-8-5.08_1x08_P5.08mm_Horizontal, symbol Connector:Screw_Terminal_01x08
- removed J7: Screw_Terminal_01x02, TerminalBlock_Phoenix:TerminalBlock_Phoenix_MKDS-1,5-2-5.08_1x02_P5.08mm_Horizontal, symbol Connector:Screw_Terminal_01x02
- removed Q1, Q10, Q2, Q3, Q4, Q5, Q6, Q7, Q8, Q9: BSS138, Package_TO_SOT_THT:TO-92L_HandSolder, symbol Transistor_FET:BSS138
- removed R10, R11, R12, R13, R14, R15, R16, R40, R41, R42, R43, R44, R45, R46, R47, R48, R49, R5, R50, R51, R52, R53, R54, R55, R6, R7, R8, R9: 560, Resistor_THT:R_Axial_DIN0204_L3.6mm_D1.6mm_P5.08mm_Horizontal, symbol Device:R
- removed R17, R18, R19, R20, R21, R22, R23, R24, R25, R26, R27, R28, R29, R30, R31, R33, R35, R36, R38, R39: 10k, Resistor_THT:R_Axial_DIN0204_L3.6mm_D1.6mm_P5.08mm_Horizontal, symbol Device:R
- removed R32, R34, R37, R56, R57, R58, R59, R60, R61, R62, R63, R64: 10K, Resistor_THT:R_Axial_DIN0204_L3.6mm_D1.6mm_P5.08mm_Horizontal, symbol Device:R
- removed SW1, SW2, SW3, SW4: SW_DIP_x03, Button_Switch_THT:SW_DIP_SPSTx03_Slide_9.78x9.8mm_W7.62mm_P2.54mm, symbol Switch:SW_DIP_x03
- removed U10, U11, U12, U13, U14, U15, U16, U17, U19, U2, U20, U21, U22, U23, U24, U25, U26, U27, U28, U29, U3, U30, U31, U32, U33, U34, U4, U5, U6, U7, U8, U9: SFH617A-1X006, Package_DIP:DIP-4_W10.16mm, symbol Isolator:SFH617A-1X006
- removed U35: MCP23017_SP, Package_DIP:DIP-28_W7.62mm, symbol Interface_Expansion:MCP23017_SP
- removed U38, U40: ULN2003A, Package_DIP:DIP-16_W7.62mm_Socket, symbol Transistor_Array:ULN2003A
- added J13, J14, J15, J16: Pin Header_01x10, Connector_PinHeader_2.54mm:PinHeader_1x10_P2.54mm_Vertical, symbol Connector:Screw_Terminal_01x10
- added J7: Screw_Terminal_01x08, TerminalBlock_Phoenix:TerminalBlock_Phoenix_MKDS-1,5-8-5.08_1x08_P5.08mm_Horizontal, symbol Connector:Screw_Terminal_01x08
- added JP1, JP2, JP3, JP4: Jumper_2_Open, Connector_PinHeader_2.54mm:PinHeader_1x02_P2.54mm_Vertical, symbol Jumper:Jumper_2_Open
- added U2: MCP23017_SP, Package_DIP:DIP-28_W7.62mm, symbol Interface_Expansion:MCP23017_SP
- added U3, U4: ULN2003A, Package_DIP:DIP-16_W7.62mm_Socket, symbol Transistor_Array:ULN2003A
- R1, R2, R3, R4: value 560 -> 10K
- U1: footprint MODULE_ESP32-DEVKITC -> footprints:MODULE_ESP32-DEVKITC
Connections:
- net I2C-SCL-5V is gone; now on an unnamed net: U18.12 (SCK), U36.12 (SCK), U37.12 (SCK)
- net I2C-SDA-5V is gone; now on an unnamed net: U18.13 (SDA), U36.13 (SDA), U37.13 (SDA)
- net +3V3: now also R1.1, R2.1, J13.1 (Pin_1), J13.10 (Pin_10), J15.1 (Pin_1), J15.10 (Pin_10); no longer J1.1 (Pin_1)
- net +5V: now also J4.1 (Pin_1), R3.1, R4.1, U18.15 (A0), U18.16 (A1), U18.17 (A2), U36.17 (A2), J14.1 (Pin_1), J16.1 (Pin_1), JP1.2 (B), JP2.2 (B), JP3.2 (B), JP4.2 (B), U2.16 (A1), U2.17 (A2), U2.9 (VDD), U3.9 (COM), U4.9 (COM); no longer J10.8 (Pin_8), J11.8 (Pin_8), J8.8 (Pin_8)
- net GND: now also J4.2 (Pin_2), U36.15 (A0), U36.16 (A1), U37.15 (A0), U37.16 (A1), U37.17 (A2), J14.10 (Pin_10), J16.10 (Pin_10), U2.10 (VSS), U2.15 (A0), U3.8 (GND), U4.8 (GND); no longer J1.2 (Pin_2), J1.3 (Pin_3), J1.4 (Pin_4), J1.5 (Pin_5)
- net at J3.7 (Pin_7): now also U18.27 (GPA6)
- net at J5.6 (Pin_6): now also U2.3 (GPB2)
- net at U18.19 (INTB): now also J16.7 (Pin_7)
- net at J3.3 (Pin_3): now also U18.23 (GPA2)
- net at U18.5 (GPB4): now also J2.5 (Pin_5)
- net at J3.4 (Pin_4): now also U18.24 (GPA3)
- net at J2.7 (Pin_7): now also U18.7 (GPB6)
- net at J5.1 (Pin_1): now also U2.8 (GPB7)
- net at J2.2 (Pin_2): now also U18.2 (GPB1); no longer R2.1
- net at R2.2: now also U1.36 (IO22), J15.3 (Pin_3)
- net at R3.2: now also J16.2 (Pin_2), U2.13 (SDA)
- net at U18.3 (GPB2): now also J2.3 (Pin_3)
- net at J3.1 (Pin_1): now also U18.21 (GPA0)
- net at J3.2 (Pin_2): now also U18.22 (GPA1)
- net at J3.5 (Pin_5): now also U18.25 (GPA4)
- net at J3.6 (Pin_6): now also U18.26 (GPA5)
- net at J3.8 (Pin_8): now also U18.28 (GPA7)
- net at U37.1 (GPB0): now also U4.5 (I5)
- net at U37.18 (~{RESET}): now also JP4.1 (A)
- net at U37.2 (GPB1): now also U4.4 (I4)
- net at U37.25 (GPA4): now also U42.4 (I4); no longer U42.1 (I1)
- net at U37.26 (GPA5): now also U42.3 (I3); no longer U42.2 (I2)
- net at U37.27 (GPA6): now also U42.2 (I2); no longer U42.3 (I3)
- net at U37.28 (GPA7): now also U42.1 (I1); no longer U42.4 (I4)
- net at U37.3 (GPB2): now also U4.3 (I3)
- net at U37.4 (GPB3): now also U4.2 (I2)
- net at U37.5 (GPB4): now also U4.1 (I1)
- net at U37.6 (GPB5): now also U41.3 (I3); no longer U41.1 (I1)
- net at U37.8 (GPB7): now also U41.1 (I1); no longer U41.3 (I3)
- net at U42.16 (O1): now also J11.5 (Pin_5)
- net at U42.15 (O2): now also J11.6 (Pin_6)
- net at U42.14 (O3): now also J11.7 (Pin_7)
- net at U42.13 (O4): now also J11.8 (Pin_8)
- net at J6.1 (Pin_1): now also U2.21 (GPA0)
- net at J6.6 (Pin_6): now also U2.26 (GPA5)
- net at J2.8 (Pin_8): now also U18.8 (GPB7)
- net at U41.10 (O7): now also J11.4 (Pin_4); no longer J11.7 (Pin_7)
- net at U41.11 (O6): now also J11.3 (Pin_3); no longer J11.6 (Pin_6)
- net at U41.12 (O5): now also J11.2 (Pin_2); no longer J11.5 (Pin_5)
- net at U41.13 (O4): now also J11.1 (Pin_1); no longer J11.4 (Pin_4)
- net at U41.14 (O3): now also J10.6 (Pin_6); no longer J11.3 (Pin_3)
- net at U41.15 (O2): now also J10.7 (Pin_7); no longer J11.2 (Pin_2)
- net at U41.16 (O1): now also J10.8 (Pin_8); no longer J11.1 (Pin_1)
- net at U18.6 (GPB5): now also J2.6 (Pin_6)
- net at J5.2 (Pin_2): now also U2.7 (GPB6)
- net at J5.3 (Pin_3): now also U2.6 (GPB5)
- net at J5.4 (Pin_4): now also U2.5 (GPB4)
- net at J5.5 (Pin_5): now also U2.4 (GPB3)
- net at J5.7 (Pin_7): now also U2.2 (GPB1)
- net at J5.8 (Pin_8): now also U2.1 (GPB0)
- net at U1.28 (IO17): now also J15.7 (Pin_7)
- net at U1.30 (IO18): now also J15.6 (Pin_6)
- net at U1.31 (IO19): now also J15.5 (Pin_5)
- net at U1.33 (IO21): now also R1.2, J15.2 (Pin_2)
- net at U1.37 (IO23): now also J15.4 (Pin_4)
- net at U39.16 (O1): now also J8.8 (Pin_8)
- net at U39.15 (O2): now also J7.8 (Pin_8)
- net at U39.14 (O3): now also J7.7 (Pin_7)
- net at U39.13 (O4): now also J7.6 (Pin_6)
- net at U39.12 (O5): now also J7.5 (Pin_5)
- net at U39.11 (O6): now also J7.4 (Pin_4)
- net at U39.10 (O7): now also J7.3 (Pin_3)
- net at U18.18 (~{RESET}): now also JP1.1 (A)
- net at J6.3 (Pin_3): now also U2.23 (GPA2)
- net at U36.27 (GPA6): now also U4.6 (I6)
- net at J10.5 (Pin_5): now also U4.16 (O1)
- net at J10.4 (Pin_4): now also U4.15 (O2)
- net at J10.3 (Pin_3): now also U4.14 (O3)
- net at J10.2 (Pin_2): now also U4.13 (O4)
- net at J10.1 (Pin_1): now also U4.12 (O5)
- net at U36.28 (GPA7): now also U4.7 (I7)
- net at U36.1 (GPB0): now also U3.7 (I7)
- net at U36.18 (~{RESET}): now also JP3.1 (A)
- net at U36.2 (GPB1): now also U3.6 (I6)
- net at U36.3 (GPB2): now also U3.5 (I5)
- net at U36.4 (GPB3): now also U3.4 (I4)
- net at U36.5 (GPB4): now also U3.3 (I3)
- net at U36.6 (GPB5): now also U3.2 (I2)
- net at U36.7 (GPB6): now also U3.1 (I1)
- net at U18.1 (GPB0): now also J2.1 (Pin_1)
- net at J6.4 (Pin_4): now also U2.24 (GPA3)
- net at U18.20 (INTA): now also J16.6 (Pin_6)
- net at U18.4 (GPB3): now also J2.4 (Pin_4)
- net at J6.2 (Pin_2): now also U2.22 (GPA1)
- net at R4.2: now also J16.3 (Pin_3), U2.12 (SCK)
- net at J6.5 (Pin_5): now also U2.25 (GPA4)
- net at J6.7 (Pin_7): now also U2.27 (GPA6)
- net at J6.8 (Pin_8): now also U2.28 (GPA7)
- net at J8.7 (Pin_7): now also U3.16 (O1)
- net at J8.6 (Pin_6): now also U3.15 (O2)
- net at J8.5 (Pin_5): now also U3.14 (O3)
- net at J8.4 (Pin_4): now also U3.13 (O4)
- net at J8.3 (Pin_3): now also U3.12 (O5)
- net at J8.2 (Pin_2): now also U3.11 (O6)
- net at J8.1 (Pin_1): now also U3.10 (O7)
- new net: J7.1 (Pin_1), U4.10 (O7)
- new net: J7.2 (Pin_2), U4.11 (O6)
- new net: JP2.1 (A), U2.18 (~{RESET})
- new net: J16.4 (Pin_4), U2.20 (INTA)
- new net: J16.5 (Pin_5), U2.19 (INTB)
- new net: J1.2 (Pin_2), J1.3 (Pin_3), J1.4 (Pin_4), J1.5 (Pin_5)
- no-connect marks 30 -> 56
Other:
- note added: "Finder Relay, 5V, Icoil = 100 mA"
- note added: "NOTE: Connector flipped for convenient layout reasons."
- note added: "UNL2003, Imax = 500 mA"
- moved on the sheet: C1, C3, C4, H1, H2, H3, H4, J1, J10, J11, J2, J4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
